Commit message: Imported upstream version '3.6.5' of 'upstream'

File: pal_gripper_description/robots/gripper_test.urdf.xacro (robot description, xacro)
@@ -18,4 +18,5 @@
   <xacro:include filename="$(find pal_gripper_description)/urdf/gripper.urdf.xacro" />
   <xacro:include filename="$(find pal_urdf_utils)/urdf/materials.urdf.xacro" />
+  <xacro:property name="gazebo_version" default="$(arg gazebo_version)"/>
   <!-- Generic simulator_gazebo plugins -->
   <!-- ros2_control -->

File: pal_gripper_description/urdf/gripper.urdf.xacro (robot description, xacro)
@@ -69,10 +69,18 @@
     <material>Gazebo/Black</material>
   </gazebo>
+  <!-- TODO: set lower limit back to 0 when moving to Gazebo Harmonic or ROS 2 Jazzy -->
+  <!-- See https://github.com/gazebosim/gz-sim/issues/1684 for more information -->
+  <xacro:if value="${gazebo_version == 'classic'}">
+    <xacro:property name="gripper_lower_limit" value="0.0"/>
+  </xacro:if>
+  <xacro:if value="${gazebo_version == 'gazebo'}">
+    <xacro:property name="gripper_lower_limit" value="-1e-3"/>
+  </xacro:if>
   <joint name="${name}_right_finger_joint" type="prismatic">
-    <origin rpy="0 0 0" xyz="0 0 0.01" />
+    <origin rpy="0 0 0" xyz="0 0 -0.01" />
     <parent link="${name}_link" />
     <child link="${name}_right_finger_link" />
     <axis xyz="1 0 0" />
-    <limit effort="16" lower="0.0" upper="0.045" velocity="0.05" />
+    <limit effort="16" lower="${gripper_lower_limit}" upper="0.045" velocity="0.05" />
     <calibration rising="0.0" />
     <dynamics damping="80" friction="2.0"/>
@@ -108,9 +116,9 @@
   </gazebo>
   <joint name="${name}_left_finger_joint" type="prismatic">
-    <origin rpy="0 0 0" xyz="0 0 0.01" />
+    <origin rpy="0 0 0" xyz="0 0 -0.01" />
     <parent link="${name}_link" />
     <child link="${name}_left_finger_link" />
     <axis xyz="-1 0 0" />
-    <limit effort="16" lower="0" upper="0.045" velocity="0.05" />
+    <limit effort="16" lower="${gripper_lower_limit}" upper="0.045" velocity="0.05" />
     <calibration rising="0.0" />
     <dynamics damping="80" friction="2.0"/>
